Commit message: making URDF ready for Gazebo.

File: gazebo_own_urdf/urdf/teslabot.urdf.xacro (robot description, xacro)
@@ -1,232 +1,887 @@
-<?xml version="1.0"?>
-<robot name="robot" xmlns:xacro="http://ros.org/wiki/xacro">
+<?xml version="1.0" encoding="utf-8"?>
+<!-- This URDF was automatically created by SolidWorks to URDF Exporter! Originally created by Stephen Brawner (brawner@gmail.com)
+     Commit Version: 1.6.0-4-g7f85cfe  Build Version: 1.6.7995.38578
+     For more information, please see http://wiki.ros.org/sw_urdf_exporter -->
+<robot
+  name="final_7dof_urdf_9oct2024" xmlns:xacro="http://ros.org/wiki/xacro">
   <link name="world"/>
-  <link name="head">
-    <inertial>
-      <mass value="1"/>
-      <inertia ixx=".1" ixy="0" ixz="0" iyy=".1" iyz="0" izz=".1" />
-    </inertial>
-    <visual>
-      <origin xyz="0 0 0" rpy="0 0 0" />
-      <geometry>
-        <!-- <cylinder radius="0.01" length=".5" /> -->
-        <mesh filename="$(find gazebo_tutorial)/meshes/head.STL" scale="1 1 1"/>
-      </geometry>
-      <material name="black">
-        <color rgba="0 0 0 1"/> <!-- Black color -->
-      </material>
-    </visual>
-  </link>
-  <joint name="world_to_head" type="fixed">
-    <origin xyz="0 0 1" />
+  <joint name="base_joint" type="fixed">
     <parent link="world"/>
-    <child link="head"/>
-  </joint>
-  <link name="body">
-    <inertial>
-      <mass value="1"/>
-      <inertia ixx=".1" ixy="0" ixz="0" iyy=".1" iyz="0" izz=".1" />
-    </inertial>
-    <visual>
-      <origin xyz="0 0 0" rpy="0 0 0" />
-      <geometry>
-        <mesh filename="$(find gazebo_tutorial)/meshes/body.STL" scale="1 1 1"/>
-      </geometry>
-      <material name="gray">
-        <color rgba=".2 .2 .2 1" />
-      </material>
-    </visual>
-  </link>
-  <joint name="head_to_body" type="fixed">
-    <origin xyz="0 0 0" />
-    <parent link="head"/>
-    <child link="body"/>
-  </joint>
-  <link name="shoulder_right">
-    <inertial>
-      <mass value="1"/>
-      <inertia ixx=".1" ixy="0" ixz="0" iyy=".1" iyz="0" izz=".1" />
-    </inertial>
-    <visual>
-      <origin xyz="0 0 0" rpy="0 0 0" />
-      <geometry>
-        <mesh filename="$(find gazebo_tutorial)/meshes/shoulder.STL" scale="1 1 1"/>
-      </geometry>
-      <material name="gray">
-        <color rgba=".2 .2 .2 1" />
-      </material>
-    </visual>
-  </link>
-  <joint name="body_to_shoulder_right" type="revolute">
-    <origin xyz="0.206 0 -0.0635" rpy="-${pi/2} 0 0"/>
-    <parent link="body"/>
-    <child link="shoulder_right"/>
-    <axis rpy="0 0 0" xyz="0 0 1"/>
-    <limit lower="-${pi}" upper="${pi}" effort="100" velocity="20"/>
-  </joint>
-  <link name="shoulder_left">
-    <inertial>
-      <mass value="1"/>
-      <inertia ixx=".1" ixy="0" ixz="0" iyy=".1" iyz="0" izz=".1" />
-    </inertial>
-    <visual>
-      <origin xyz="0 0 0" rpy="0 0 0" />
-      <geometry>
-        <mesh filename="$(find gazebo_tutorial)/meshes/shoulder.STL" scale="1 1 1"/>
-      </geometry>
-      <material name="gray">
-        <color rgba=".2 .2 .2 1" />
-      </material>
-    </visual>
-  </link>
-  <joint name="body_to_shoulder_left" type="revolute">
-    <origin xyz="-0.206 0 -0.0635" rpy="${pi/2} 0 ${pi}"/>
-    <parent link="body"/>
-    <child link="shoulder_left"/>
-    <axis rpy="0 0 0" xyz="0 0 1"/>
-    <limit lower="-${pi}" upper="${pi}" effort="100" velocity="20"/>
-  </joint>
-  <link name="arm_upper_right">
-    <inertial>
-      <mass value="1"/>
-      <inertia ixx=".1" ixy="0" ixz="0" iyy=".1" iyz="0" izz=".1" />
-    </inertial>
-    <visual>
-      <origin xyz="0 0 0" rpy="0 0 0" />
-      <geometry>
-        <mesh filename="$(find gazebo_tutorial)/meshes/arm_upper.STL" scale="1 1 1"/>
-      </geometry>
-      <material name="gray">
-        <color rgba=".2 .2 .2 1" />
-      </material>
-    </visual>
-  </link>
-  <joint name="shoulder_to_arm_upper_right" type="revolute">
-    <origin xyz="0 0 0" rpy="0 0 ${pi}"/>
-    <parent link="shoulder_right"/>
-    <child link="arm_upper_right"/>
-    <axis rpy="0 0 0" xyz="0 0 1"/>
-    <limit lower="-${pi}" upper="${pi}" effort="100" velocity="20"/>
-  </joint>
-  <link name="arm_upper_left">
-    <inertial>
-      <mass value="1"/>
-      <inertia ixx=".1" ixy="0" ixz="0" iyy=".1" iyz="0" izz=".1" />
-    </inertial>
-    <visual>
-      <origin xyz="0 0 0" rpy="0 0 0" />
-      <geometry>
-        <mesh filename="$(find gazebo_tutorial)/meshes/arm_upper.STL" scale="1 1 1"/>
-      </geometry>
-      <material name="gray">
-        <color rgba=".2 .2 .2 1" />
-      </material>
-    </visual>
-  </link>
-  <joint name="shoulder_to_arm_upper_left" type="revolute">
-    <origin xyz="0 0 0" rpy="0 0 0"/>
-    <parent link="shoulder_left"/>
-    <child link="arm_upper_left"/>
-    <axis rpy="0 0 0" xyz="0 0 1"/>
-    <limit lower="-${pi}" upper="${pi}" effort="100" velocity="20"/>
-  </joint>
-  <link name="arm_lower_right">
-    <inertial>
-      <mass value="1"/>
-      <inertia ixx=".1" ixy="0" ixz="0" iyy=".1" iyz="0" izz=".1" />
-    </inertial>
-    <visual>
-      <origin xyz="0 0 0" rpy="0 0 0" />
-      <geometry>
-        <mesh filename="$(find gazebo_tutorial)/meshes/arm_lower.STL" scale="1 1 1"/>
-      </geometry>
-      <material name="gray">
-        <color rgba=".2 .2 .2 1" />
-      </material>
-    </visual>
-  </link>
-  <joint name="arm_upper_to_lower_right" type="revolute">
-    <origin xyz="0 -.358 0" rpy="0 -${pi/2} 0"/>
-    <parent link="arm_upper_right"/>
-    <child link="arm_lower_right"/>
-    <axis rpy="0 0 0" xyz="0 0 1"/>
-    <limit lower="-${pi}" upper="${pi}" effort="100" velocity="20"/>
-  </joint>
-  <link name="arm_lower_left">
-    <inertial>
-      <mass value="1"/>
-      <inertia ixx=".1" ixy="0" ixz="0" iyy=".1" iyz="0" izz=".1" />
-    </inertial>
-    <visual>
-      <origin xyz="0 0 0" rpy="0 0 0" />
-      <geometry>
-        <mesh filename="$(find gazebo_tutorial)/meshes/arm_lower.STL" scale="1 1 1"/>
-      </geometry>
-      <material name="gray">
-        <color rgba=".2 .2 .2 1" />
-      </material>
-    </visual>
-  </link>
-  <joint name="arm_upper_to_lower_left" type="revolute">
-    <origin xyz="0 -.358 0" rpy="0 ${pi/2} 0"/>
-    <parent link="arm_upper_left"/>
-    <child link="arm_lower_left"/>
-    <axis rpy="0 0 0" xyz="0 0 1"/>
-    <limit lower="-${pi}" upper="${pi}" effort="100" velocity="20"/>
-  </joint>
-  <link name="hand_right">
-    <inertial>
-      <mass value="1"/>
-      <inertia ixx=".1" ixy="0" ixz="0" iyy=".1" iyz="0" izz=".1" />
-    </inertial>
-    <visual>
-      <origin xyz="0 0 0" rpy="0 0 0" />
-      <geometry>
-        <mesh filename="$(find gazebo_tutorial)/meshes/hand_right.STL" scale="1 1 1"/>
-      </geometry>
-      <material name="gray">
-        <color rgba=".2 .2 .2 1" />
-      </material>
-    </visual>
-  </link>
-  <joint name="arm_lower_to_hand_right" type="fixed">
-    <origin xyz="0 -.338 0" rpy="${pi/2} -${pi} 0"/>
-    <parent link="arm_lower_right"/>
-    <child link="hand_right"/>
-  </joint>
-  <link name="hand_left">
-    <inertial>
-      <mass value="1"/>
-      <inertia ixx=".1" ixy="0" ixz="0" iyy=".1" iyz="0" izz=".1" />
-    </inertial>
-    <visual>
-      <origin xyz="0 0 0" rpy="0 0 0" />
-      <geometry>
-        <mesh filename="$(find gazebo_tutorial)/meshes/hand_left.STL" scale="1 1 1"/>
-      </geometry>
-      <material name="gray">
-        <color rgba=".2 .2 .2 1" />
-      </material>
-    </visual>
-  </link>
-  <joint name="arm_lower_to_hand_left" type="fixed">
-    <origin xyz="0 -.338 0" rpy="${pi/2} 0 0"/>
-    <parent link="arm_lower_left"/>
-    <child link="hand_left"/>
-  </joint>
-  <gazebo reference="head">
-    <material>Gazebo/Black</material>
-  </gazebo>
-  <gazebo reference="body">
-    <material>Gazebo/White</material>
-  </gazebo>
+    <child link="base_link"/>
+    <origin rpy="0 0 0" xyz="-0.081136 0.15 -0.051"/>
+    </joint>
+  <link
+    name="base_link">
+    <inertial>
+      <origin
+        xyz="0.00049737 0.00026123 0.0072038"
+        rpy="0 0 0" />
+      <mass
+        value="6.9112" />
+      <inertia
+        ixx="0.046617"
+        ixy="0.00010077"
+        ixz="5.1488E-08"
+        iyy="0.046482"
+        iyz="-1.4461E-07"
+        izz="0.092984" />
+    </inertial>
+    <visual>
+      <origin
+        xyz="0 0 0"
+        rpy="0 0 0" />
+      <geometry>
+        <mesh
+          filename="package://final_7dof_urdf_9oct2024/meshes/base_link.STL" />
+      </geometry>
+      <material
+        name="">
+        <color
+          rgba="0.77647 0.75686 0.73725 1" />
+      </material>
+    </visual>
+    <collision>
+      <origin
+        xyz="0 0 0"
+        rpy="0 0 0" />
+      <geometry>
+        <mesh
+          filename="package://final_7dof_urdf_9oct2024/meshes/base_link.STL" />
+      </geometry>
+    </collision>
+  </link>
+  <link
+    name="Link_1">
+    <inertial>
+      <origin
+        xyz="1.4551E-05 -0.0043711 0.069929"
+        rpy="0 0 0" />
+      <mass
+        value="1.4053" />
+      <inertia
+        ixx="0.0017174"
+        ixy="6.6784E-08"
+        ixz="3.5551E-07"
+        iyy="0.002626"
+        iyz="6.0024E-06"
+        izz="0.0017063" />
+    </inertial>
+    <visual>
+      <origin
+        xyz="0 0 0"
+        rpy="0 0 0" />
+      <geometry>
+        <mesh
+          filename="package://final_7dof_urdf_9oct2024/meshes/Link_1.STL" />
+      </geometry>
+      <material
+        name="">
+        <color
+          rgba="0 0 0 1" />
+      </material>
+    </visual>
+    <collision>
+      <origin
+        xyz="0 0 0"
+        rpy="0 0 0" />
+      <geometry>
+        <mesh
+          filename="package://final_7dof_urdf_9oct2024/meshes/Link_1.STL" />
+      </geometry>
+    </collision>
+  </link>
+  <joint
+    name="joint_1"
+    type="continuous">
+    <origin
+      xyz="0 0 0.05"
+      rpy="0 0 3.1416" />
+    <parent
+      link="base_link" />
+    <child
+      link="Link_1" />
+    <axis
+      xyz="0 0 -1" />
+    <limit
+      lower="0"
+      upper="3.14"
+      effort="0"
+      velocity="0" />
+  </joint>
+  <link
+    name="Link_2">
+    <inertial>
+      <origin
+        xyz="-6.5548E-05 0.21409 0.034291"
+        rpy="0 0 0" />
+      <mass
+        value="3.4329" />
+      <inertia
+        ixx="0.0091312"
+        ixy="-2.4753E-06"
+        ixz="8.4256E-07"
+        iyy="0.0057112"
+        iyz="5.0607E-06"
+        izz="0.0099035" />
+    </inertial>
+    <visual>
+      <origin
+        xyz="0 0 0"
+        rpy="0 0 0" />
+      <geometry>
+        <mesh
+          filename="package://final_7dof_urdf_9oct2024/meshes/Link_2.STL" />
+      </geometry>
+      <material
+        name="">
+        <color
+          rgba="1 1 1 1" />
+      </material>
+    </visual>
+    <collision>
+      <origin
+        xyz="0 0 0"
+        rpy="0 0 0" />
+      <geometry>
+        <mesh
+          filename="package://final_7dof_urdf_9oct2024/meshes/Link_2.STL" />
+      </geometry>
+    </collision>
+  </link>
+  <joint
+    name="joint_2"
+    type="revolute">
+    <origin
+      xyz="0 -0.02999999999948 0.107500000000395"
+      rpy="1.5707963267949 0 -3.14159265358979" />
+    <parent
+      link="Link_1" />
+    <child
+      link="Link_2" />
+    <axis
+      xyz="0 0 -1" />
+    <limit
+      lower="-1.9199"
+      upper="1.9199"
+      effort="0"
+      velocity="0" />
+  </joint>
+  <link
+    name="Link_3">
+    <inertial>
+      <origin
+        xyz="-2.1655E-05 0.0044003 0.0672"
+        rpy="0 0 0" />
+      <mass
+        value="1.3788" />
+      <inertia
+        ixx="0.0016215"
+        ixy="-9.275E-08"
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