Commit message: changed the coordinates to default 0,0,0

File: gazebo_own_urdf/urdf/final_7dof_urdf_9oct2024.urdf.xacro (robot description, xacro)
@@ -1,3 +1,3 @@
-<?xml version="1.0" encoding="utf-8"?>
+<?xml version="1.0"?>
 <!-- This URDF was automatically created by SolidWorks to URDF Exporter! Originally created by Stephen Brawner (brawner@gmail.com)
      Commit Version: 1.6.0-4-g7f85cfe  Build Version: 1.6.7995.38578
@@ -9,5 +9,5 @@
     <parent link="world"/>
     <child link="base_link"/>
-    <origin rpy="0 0 0" xyz="-0.081136 0.15 -0.051"/>
+    <origin rpy="0 0 0" xyz="0 0 0"/>
     </joint>
   <link

File: install/gazebo_own_urdf/share/gazebo_own_urdf/urdf/final_7dof_urdf_9oct2024.urdf.xacro (robot description, xacro)
@@ -9,5 +9,5 @@
     <parent link="world"/>
     <child link="base_link"/>
-    <origin rpy="0 0 0" xyz="-0.081136 0.15 -0.051"/>
+    <origin rpy="0 0 0" xyz="0 0 0"/>
     </joint>
   <link

Commit message: reverted the changes in urdf (xml tag + base joint location)

File: gazebo_own_urdf/urdf/final_7dof_urdf_9oct2024.urdf.xacro (robot description, xacro)
@@ -1,3 +1,3 @@
-<?xml version="1.0"?>
+<?xml version="1.0" encoding="utf-8"?>
 <!-- This URDF was automatically created by SolidWorks to URDF Exporter! Originally created by Stephen Brawner (brawner@gmail.com)
      Commit Version: 1.6.0-4-g7f85cfe  Build Version: 1.6.7995.38578
@@ -9,5 +9,5 @@
     <parent link="world"/>
     <child link="base_link"/>
-    <origin rpy="0 0 0" xyz="0 0 0"/>
+    <origin rpy="0 0 0" xyz=""-0.081136 0.15 -0.051""/>
     </joint>
   <link

Commit message: urdf errors.

File: gazebo_own_urdf/urdf/final_7dof_urdf_9oct2024.urdf.xacro (robot description, xacro)
@@ -9,5 +9,5 @@
     <parent link="world"/>
     <child link="base_link"/>
-    <origin rpy="0 0 0" xyz=""-0.081136 0.15 -0.051""/>
+    <origin rpy="0 0 0" xyz="-0.081136 0.15 -0.051"/>
     </joint>
   <link

File: install/gazebo_own_urdf/share/gazebo_own_urdf/urdf/final_7dof_urdf_9oct2024.urdf.xacro (robot description, xacro)
@@ -9,5 +9,5 @@
     <parent link="world"/>
     <child link="base_link"/>
-    <origin rpy="0 0 0" xyz="0 0 0"/>
+    <origin rpy="0 0 0" xyz=""-0.081136 0.15 -0.051""/>
     </joint>
   <link

Commit message: Removed the <!-- This URDF was....> comment from URDF as it was causing this error: Parser Error Couldn't parse parameter override rule...

File: gazebo_own_urdf/urdf/final_7dof_urdf_9oct2024.urdf.xacro (robot description, xacro)
@@ -1,6 +1,3 @@
-<?xml version="1.0" encoding="utf-8"?>
-<!-- This URDF was automatically created by SolidWorks to URDF Exporter! Originally created by Stephen Brawner (brawner@gmail.com)
-     Commit Version: 1.6.0-4-g7f85cfe  Build Version: 1.6.7995.38578
-     For more information, please see http://wiki.ros.org/sw_urdf_exporter -->
+<?xml version="1.0"?>
 <robot
   name="final_7dof_urdf_9oct2024" xmlns:xacro="http://ros.org/wiki/xacro">
@@ -9,5 +6,5 @@
     <parent link="world"/>
     <child link="base_link"/>
-    <origin rpy="0 0 0" xyz="-0.081136 0.15 -0.051"/>
+    <origin rpy="0 0 0" xyz="0 0 0"/>
     </joint>
   <link

File: install/gazebo_own_urdf/share/gazebo_own_urdf/urdf/final_7dof_urdf_9oct2024.urdf.xacro (robot description, xacro)
@@ -1,6 +1,3 @@
-<?xml version="1.0" encoding="utf-8"?>
-<!-- This URDF was automatically created by SolidWorks to URDF Exporter! Originally created by Stephen Brawner (brawner@gmail.com)
-     Commit Version: 1.6.0-4-g7f85cfe  Build Version: 1.6.7995.38578
-     For more information, please see http://wiki.ros.org/sw_urdf_exporter -->
+<?xml version="1.0"?>
 <robot
   name="final_7dof_urdf_9oct2024" xmlns:xacro="http://ros.org/wiki/xacro">
@@ -9,5 +6,5 @@
     <parent link="world"/>
     <child link="base_link"/>
-    <origin rpy="0 0 0" xyz=""-0.081136 0.15 -0.051""/>
+    <origin rpy="0 0 0" xyz="0 0 0"/>
     </joint>
   <link
