Commit message: random joint angles for each time step.

File: install/gazebo_own_urdf/share/gazebo_own_urdf/urdf/final_7dof_urdf_9oct2024.urdf.xacro (robot description, xacro)
@@ -1,950 +1 @@
-<?xml version="1.0"?>
-<robot
-  name="final_7dof_urdf_9oct2024" xmlns:xacro="http://ros.org/wiki/xacro">
-  <link name="world"/>
-  <joint name="base_joint" type="fixed">
-    <parent link="world"/>
-    <child link="base_link"/>
-    <origin rpy="0 0 0" xyz="0 0 0"/>
-    </joint>
-  <link
-    name="base_link">
-    <inertial>
-      <origin
-        xyz="0.00049737 0.00026123 0.0072038"
-        rpy="0 0 0" />
-      <mass
-        value="6.9112" />
-      <inertia
-        ixx="0.046617"
-        ixy="0.00010077"
-        ixz="5.1488E-08"
-        iyy="0.046482"
-        iyz="-1.4461E-07"
-        izz="0.092984" />
-    </inertial>
-    <visual>
-      <origin
-        xyz="0 0 0"
-        rpy="0 0 0" />
-      <geometry>
-        <mesh
-          filename="$(find gazebo_own_urdf)/meshes/base_link.STL" />
-      </geometry>
-      <material
-        name="">
-        <color
-          rgba="0.77647 0.75686 0.73725 1" />
-      </material>
-    </visual>
-    <collision>
-      <origin
-        xyz="0 0 0"
-        rpy="0 0 0" />
-      <geometry>
-        <mesh
-          filename="$(find gazebo_own_urdf)/meshes/base_link.STL" />
-      </geometry>
-    </collision>
-  </link>
-  <link
-    name="Link_1">
-    <inertial>
-      <origin
-        xyz="1.4551E-05 -0.0043711 0.069929"
-        rpy="0 0 0" />
-      <mass
-        value="1.4053" />
-      <inertia
-        ixx="0.0017174"
-        ixy="6.6784E-08"
-        ixz="3.5551E-07"
-        iyy="0.002626"
-        iyz="6.0024E-06"
-        izz="0.0017063" />
-    </inertial>
-    <visual>
-      <origin
-        xyz="0 0 0"
-        rpy="0 0 0" />
-      <geometry>
-        <mesh
-          filename="$(find gazebo_own_urdf)/meshes/Link_1.STL" />
-      </geometry>
-      <material
-        name="">
-        <color
-          rgba="0 0 0 1" />
-      </material>
-    </visual>
-    <collision>
-      <origin
-        xyz="0 0 0"
-        rpy="0 0 0" />
-      <geometry>
-        <mesh
-          filename="$(find gazebo_own_urdf)/meshes/Link_1.STL" />
-      </geometry>
-    </collision>
-  </link>
-  <joint
-    name="joint_1"
-    type="continuous">
-    <origin
-      xyz="0 0 0.05"
-      rpy="0 0 3.1416" />
-    <parent
-      link="base_link" />
-    <child
-      link="Link_1" />
-    <axis
-      xyz="0 0 -1" />
-    <limit
-      lower="0"
-      upper="3.14"
-      effort="0"
-      velocity="0" />
-  </joint>
-  <link
-    name="Link_2">
-    <inertial>
-      <origin
-        xyz="-6.5548E-05 0.21409 0.034291"
-        rpy="0 0 0" />
-      <mass
-        value="3.4329" />
-      <inertia
-        ixx="0.0091312"
-        ixy="-2.4753E-06"
-        ixz="8.4256E-07"
-        iyy="0.0057112"
-        iyz="5.0607E-06"
-        izz="0.0099035" />
-    </inertial>
-    <visual>
-      <origin
-        xyz="0 0 0"
-        rpy="0 0 0" />
-      <geometry>
-        <mesh
-          filename="$(find gazebo_own_urdf)/meshes/Link_2.STL" />
-      </geometry>
-      <material
-        name="">
-        <color
-          rgba="1 1 1 1" />
-      </material>
-    </visual>
-    <collision>
-      <origin
-        xyz="0 0 0"
-        rpy="0 0 0" />
-      <geometry>
-        <mesh
-          filename="$(find gazebo_own_urdf)/meshes/Link_2.STL" />
-      </geometry>
-    </collision>
-  </link>
-  <joint
-    name="joint_2"
-    type="revolute">
-    <origin
-      xyz="0 -0.02999999999948 0.107500000000395"
-      rpy="1.5707963267949 0 -3.14159265358979" />
-    <parent
-      link="Link_1" />
-    <child
-      link="Link_2" />
-    <axis
-      xyz="0 0 -1" />
-    <limit
-      lower="-1.9199"
-      upper="1.9199"
-      effort="0"
-      velocity="0" />
-  </joint>
-  <link
-    name="Link_3">
-    <inertial>
-      <origin
-        xyz="-2.1655E-05 0.0044003 0.0672"
-        rpy="0 0 0" />
-      <mass
-        value="1.3788" />
-      <inertia
-        ixx="0.0016215"
-        ixy="-9.275E-08"
-        ixz="2.8899E-07"
-        iyy="0.0025027"
-        iyz="-5.4475E-06"
-        izz="0.0016785" />
-    </inertial>
-    <visual>
-      <origin
-        xyz="0 0 0"
-        rpy="0 0 0" />
-      <geometry>
-        <mesh
-          filename="$(find gazebo_own_urdf)/meshes/Link_3.STL" />
-      </geometry>
-      <material
-        name="">
-        <color
-          rgba="0 0 0 1" />
-      </material>
-    </visual>
-    <collision>
-      <origin
-        xyz="0 0 0"
-        rpy="0 0 0" />
-      <geometry>
-        <mesh
-          filename="$(find gazebo_own_urdf)/meshes/Link_3.STL" />
-      </geometry>
-    </collision>
-  </link>
-  <joint
-    name="joint_3"
-    type="continuous">
-    <origin
-      xyz="0.000359289684152012 0.435033961918617 0.0294474762975983"
-      rpy="1.57079632680726 0 3.14159265358979" />
-    <parent
-      link="Link_2" />
-    <child
-      link="Link_3" />
-    <axis
-      xyz="0 0 -1" />
-    <limit
-      lower="0"
-      upper="3.14"
-      effort="0"
-      velocity="0" />
-  </joint>
-  <link
-    name="Link_4">
-    <inertial>
-      <origin
-        xyz="0.22054 0.00021752 -0.034312"
-        rpy="0 0 0" />
-      <mass
-        value="3.5515" />
-      <inertia
-        ixx="0.0043885"
-        ixy="2.6288E-06"
-        ixz="-3.6827E-06"
-        iyy="0.0083524"
-        iyz="-3.8569E-06"
-        izz="0.0091315" />
-    </inertial>
-    <visual>
-      <origin
-        xyz="0 0 0"
-        rpy="0 0 0" />
-      <geometry>
-        <mesh
-          filename="$(find gazebo_own_urdf)/meshes/Link_4.STL" />
-      </geometry>
-      <material
-        name="">
-        <color
-          rgba="1 1 1 1" />
-      </material>
-    </visual>
-    <collision>
-      <origin
-        xyz="0 0 0"
-        rpy="0 0 0" />
-      <geometry>
-        <mesh
-          filename="$(find gazebo_own_urdf)/meshes/Link_4.STL" />
-      </geometry>
-    </collision>
-  </link>
-  <joint
-    name="joint_4"
-    type="revolute">
-    <origin
-      xyz="0 0.0299999999999995 0.102500000000001"
-      rpy="1.5707963267949 0 3.14159265358979" />
-    <parent
-      link="Link_3" />
-    <child
-      link="Link_4" />
-    <axis
-      xyz="0 0 1" />
-    <limit
-      lower="-0.2618"
-      upper="3.4907"
-      effort="0"
-      velocity="0" />
-  </joint>
-  <link
-    name="Link_5">
-    <inertial>
-      <origin
-        xyz="0.0058409 -0.0002627 0.054755"
-        rpy="0 0 0" />
-      <mass
-        value="1.4559" />
-      <inertia
-        ixx="0.0013388"
-        ixy="-2.389E-05"
-        ixz="-1.7038E-06"
-        iyy="0.00084376"
-        iyz="-2.3795E-07"
-        izz="0.0009966" />
-    </inertial>
-    <visual>
-      <origin
-        xyz="0 0 0"
-        rpy="0 0 0" />
-      <geometry>
-        <mesh
-          filename="$(find gazebo_own_urdf)/meshes/Link_5.STL" />
-      </geometry>
-      <material
-        name="">
-        <color
-          rgba="0 0 0 1" />
-      </material>
-    </visual>
-    <collision>
-      <origin
-        xyz="0 0 0"
-        rpy="0 0 0" />
-      <geometry>
-        <mesh
-          filename="$(find gazebo_own_urdf)/meshes/Link_5.STL" />
-      </geometry>
-    </collision>
-  </link>
-  <joint
-    name="joint_5"
-    type="continuous">
-    <origin
-      xyz="0.419299903678905 0 -0.0294999999999992"
-      rpy="0 1.5707963267949 0" />
-    <parent
-      link="Link_4" />
-    <child
-      link="Link_5" />
-    <axis
-      xyz="0 0 -1" />
-    <limit
-      lower="0"
-      upper="3.14"
-      effort="0"
-      velocity="0" />
-  </joint>
-  <link
-    name="link_6">
-    <inertial>
-      <origin
-        xyz="0.00011175 -0.056394 -0.023876"
-        rpy="0 0 0" />
-      <mass
-        value="1.4077" />
-      <inertia
-        ixx="0.00078211"
-        ixy="-9.9306E-07"
-        ixz="3.1036E-06"
-        iyy="0.0010474"
-        iyz="1.657E-06"
-        izz="0.00099212" />
-    </inertial>
-    <visual>
-      <origin
-        xyz="0 0 0"
-        rpy="0 0 0" />
-      <geometry>
-        <mesh
-          filename="$(find gazebo_own_urdf)/meshes/link_6.STL" />
-      </geometry>
-      <material
-        name="">
-        <color
-          rgba="1 1 1 1" />
-      </material>
-    </visual>
-    <collision>
-      <origin
-        xyz="0 0 0"
-        rpy="0 0 0" />
-      <geometry>
-        <mesh
-          filename="$(find gazebo_own_urdf)/meshes/link_6.STL" />
-      </geometry>
-    </collision>
-  </link>
-  <joint
-    name="joint_6"
-    type="revolute">
-    <origin
-      xyz="0.0239691789943203 -0.00121612576549357 0.0675000000000011"
-      rpy="0.0506935943659278 1.5707963267949 0" />
-    <parent
-      link="Link_5" />
-    <child
-      link="link_6" />
-    <axis
-      xyz="0 0 1" />
-    <limit
-      lower="-3.14"
-      upper="0"
-      effort="0"
-      velocity="0" />
-  </joint>
-  <link
-    name="Link_7">
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