Commit message: Removed extra joints and links.

File: gazebo_2_sim/urdf/link2_urdf.urdf.xacro (robot description, xacro)
@@ -164,715 +164,4 @@
       velocity="0" />
   </joint>
-  <link
-    name="Link_3">
-    <inertial>
-      <origin
-        xyz="-2.1655E-05 0.0044003 0.0672"
-        rpy="0 0 0" />
-      <mass
-        value="1.3788" />
-      <inertia
-        ixx="0.0016215"
-        ixy="-9.275E-08"
-        ixz="2.8899E-07"
-        iyy="0.0025027"
-        iyz="-5.4475E-06"
-        izz="0.0016785" />
-    </inertial>
-    <visual>
-      <origin
-        xyz="0 0 0"
-        rpy="0 0 0" />
-      <geometry>
-        <mesh
-          filename="$(find gazebo_own_urdf)/meshes/Link_3.STL" />
-      </geometry>
-      <material
-        name="">
-        <color
-          rgba="0 0 0 1" />
-      </material>
-    </visual>
-    <collision>
-      <origin
-        xyz="0 0 0"
-        rpy="0 0 0" />
-      <geometry>
-        <mesh
-          filename="$(find gazebo_own_urdf)/meshes/Link_3.STL" />
-      </geometry>
-    </collision>
-  </link>
-  <joint
-    name="joint_3"
-    type="continuous">
-    <origin
-      xyz="0.000359289684152012 0.435033961918617 0.0294474762975983"
-      rpy="1.57079632680726 0 3.14159265358979" />
-    <parent
-      link="Link_2" />
-    <child
-      link="Link_3" />
-    <axis
-      xyz="0 0 -1" />
-    <limit
-      lower="0"
-      upper="3.14"
-      effort="0"
-      velocity="0" />
-  </joint>
-  <link
-    name="Link_4">
-    <inertial>
-      <origin
-        xyz="0.22054 0.00021752 -0.034312"
-        rpy="0 0 0" />
-      <mass
-        value="3.5515" />
-      <inertia
-        ixx="0.0043885"
-        ixy="2.6288E-06"
-        ixz="-3.6827E-06"
-        iyy="0.0083524"
-        iyz="-3.8569E-06"
-        izz="0.0091315" />
-    </inertial>
-    <visual>
-      <origin
-        xyz="0 0 0"
-        rpy="0 0 0" />
-      <geometry>
-        <mesh
-          filename="$(find gazebo_own_urdf)/meshes/Link_4.STL" />
-      </geometry>
-      <material
-        name="">
-        <color
-          rgba="1 1 1 1" />
-      </material>
-    </visual>
-    <collision>
-      <origin
-        xyz="0 0 0"
-        rpy="0 0 0" />
-      <geometry>
-        <mesh
-          filename="$(find gazebo_own_urdf)/meshes/Link_4.STL" />
-      </geometry>
-    </collision>
-  </link>
-  <joint
-    name="joint_4"
-    type="revolute">
-    <origin
-      xyz="0 0.0299999999999995 0.102500000000001"
-      rpy="1.5707963267949 0 3.14159265358979" />
-    <parent
-      link="Link_3" />
-    <child
-      link="Link_4" />
-    <axis
-      xyz="0 0 1" />
-    <limit
-      lower="-0.2618"
-      upper="3.4907"
-      effort="0"
-      velocity="0" />
-  </joint>
-  <link
-    name="Link_5">
-    <inertial>
-      <origin
-        xyz="0.0058409 -0.0002627 0.054755"
-        rpy="0 0 0" />
-      <mass
-        value="1.4559" />
-      <inertia
-        ixx="0.0013388"
-        ixy="-2.389E-05"
-        ixz="-1.7038E-06"
-        iyy="0.00084376"
-        iyz="-2.3795E-07"
-        izz="0.0009966" />
-    </inertial>
-    <visual>
-      <origin
-        xyz="0 0 0"
-        rpy="0 0 0" />
-      <geometry>
-        <mesh
-          filename="$(find gazebo_own_urdf)/meshes/Link_5.STL" />
-      </geometry>
-      <material
-        name="">
-        <color
-          rgba="0 0 0 1" />
-      </material>
-    </visual>
-    <collision>
-      <origin
-        xyz="0 0 0"
-        rpy="0 0 0" />
-      <geometry>
-        <mesh
-          filename="$(find gazebo_own_urdf)/meshes/Link_5.STL" />
-      </geometry>
-    </collision>
-  </link>
-  <joint
-    name="joint_5"
-    type="continuous">
-    <origin
-      xyz="0.419299903678905 0 -0.0294999999999992"
-      rpy="0 1.5707963267949 0" />
-    <parent
-      link="Link_4" />
-    <child
-      link="Link_5" />
-    <axis
-      xyz="0 0 -1" />
-    <limit
-      lower="0"
-      upper="3.14"
-      effort="0"
-      velocity="0" />
-  </joint>
-  <link
-    name="link_6">
-    <inertial>
-      <origin
-        xyz="0.00011175 -0.056394 -0.023876"
-        rpy="0 0 0" />
-      <mass
-        value="1.4077" />
-      <inertia
-        ixx="0.00078211"
-        ixy="-9.9306E-07"
-        ixz="3.1036E-06"
-        iyy="0.0010474"
-        iyz="1.657E-06"
-        izz="0.00099212" />
-    </inertial>
-    <visual>
-      <origin
-        xyz="0 0 0"
-        rpy="0 0 0" />
-      <geometry>
-        <mesh
-          filename="$(find gazebo_own_urdf)/meshes/link_6.STL" />
-      </geometry>
-      <material
-        name="">
-        <color
-          rgba="1 1 1 1" />
-      </material>
-    </visual>
-    <collision>
-      <origin
-        xyz="0 0 0"
-        rpy="0 0 0" />
-      <geometry>
-        <mesh
-          filename="$(find gazebo_own_urdf)/meshes/link_6.STL" />
-      </geometry>
-    </collision>
-  </link>
-  <joint
-    name="joint_6"
-    type="revolute">
-    <origin
-      xyz="0.0239691789943203 -0.00121612576549357 0.0675000000000011"
-      rpy="0.0506935943659278 1.5707963267949 0" />
-    <parent
-      link="Link_5" />
-    <child
-      link="link_6" />
-    <axis
-      xyz="0 0 1" />
-    <limit
-      lower="-3.14"
-      upper="0"
-      effort="0"
-      velocity="0" />
-  </joint>
-  <link
-    name="Link_7">
-    <inertial>
-      <origin
-        xyz="8.2711E-06 3.9121E-07 0.0087604"
-        rpy="0 0 0" />
-      <mass
-        value="0.18439" />
-      <inertia
-        ixx="8.0523E-05"
-        ixy="-8.9234E-11"
-        ixz="-4.712E-11"
-        iyy="8.0525E-05"
-        iyz="-2.2287E-12"
-        izz="0.00015908" />
-    </inertial>
-    <visual>
-      <origin
-        xyz="0 0 0"
-        rpy="0 0 0" />
-      <geometry>
-        <mesh
-          filename="$(find gazebo_own_urdf)/meshes/Link_7.STL" />
-      </geometry>
-      <material
-        name="">
-        <color
-          rgba="0 0 0 1" />
-      </material>
-    </visual>
-    <collision>
-      <origin
-        xyz="0 0 0"
-        rpy="0 0 0" />
-      <geometry>
-        <mesh
-          filename="$(find gazebo_own_urdf)/meshes/Link_7.STL" />
-      </geometry>
-    </collision>
-  </link>
-  <joint
-    name="joint_7"
-    type="continuous">
-    <origin
-      xyz="0 -0.0909999036788988 -0.0244999999999991"
-      rpy="-1.5707963267949 0 3.14159265358979" />
-    <parent
-      link="link_6" />
-    <child
-      link="Link_7" />
-    <axis
-      xyz="0 0 -1" />
-    <limit
-      lower="0"
-      upper="3.14"
-      effort="0"
-      velocity="0" />
-  </joint>
-  <link
-    name="endeffector">
-    <inertial>
-      <origin
-        xyz="-0.0198 -0.019334 0.047383"
-        rpy="0 0 0" />
-      <mass
-        value="0.10291" />
-      <inertia
-        ixx="1.41E-05"
-        ixy="-4.3343E-07"
-        ixz="-9.812E-08"
-        iyy="2.056E-05"
-        iyz="-4.6453E-09"
-        izz="2.527E-05" />
-    </inertial>
-    <visual>
-      <origin
-        xyz="0 0 0"
-        rpy="0 0 0" />
-      <geometry>
-        <mesh
-          filename="$(find gazebo_own_urdf)/meshes/endeffector.STL" />
-      </geometry>
-      <material
-        name="">
-        <color
-          rgba="1 1 1 1" />
-      </material>
-    </visual>
-    <collision>
-      <origin
-        xyz="0 0 0"
-        rpy="0 0 0" />
-      <geometry>
-        <mesh
-          filename="$(find gazebo_own_urdf)/meshes/endeffector.STL" />
-      </geometry>
-    </collision>
-  </link>
-  <joint
-    name="endeffector"
-    type="fixed">
-    <origin
-      xyz="0 0 0"
-      rpy="0 0 0" />
-    <parent
-      link="Link_7" />
-    <child
-      link="endeffector" />
-    <axis
-      xyz="0 0 0" />
-  </joint>
-  <link
-    name="gear1">
-    <inertial>
-      <origin
-        xyz="0.00049542 -0.0057094 0.0018167"
-        rpy="0 0 0" />
-      <mass
-        value="0.0053" />
-      <inertia
-        ixx="7.5591E-07"
-        ixy="-2.1833E-08"
-        ixz="-6.9871E-09"
-        iyy="1.8107E-07"
-        iyz="3.6804E-08"
-        izz="9.2464E-07" />
-    </inertial>
-    <visual>
-      <origin
-        xyz="0 0 0"
-        rpy="0 0 0" />
-      <geometry>
-        <mesh
-          filename="$(find gazebo_own_urdf)/meshes/gear1.STL" />
-      </geometry>
-      <material
-        name="">
-        <color
-          rgba="0 0 0 1" />
-      </material>
-    </visual>
-    <collision>
-      <origin
-        xyz="0 0 0"
-        rpy="0 0 0" />
-      <geometry>
-        <mesh
-          filename="$(find gazebo_own_urdf)/meshes/gear1.STL" />
-      </geometry>
-    </collision>
-  </link>
-  <joint
-    name="gear1_joint"
-    type="revolute">
-    <origin
-      xyz="-0.0136030394768413 0.00185938617586617 0.0481789689084899"
-      rpy="-1.52010273242897 0 0" />
-    <parent
-      link="endeffector" />
-    <child
-      link="gear1" />
-    <axis
-      xyz="-0.0472460759822869 0.0506152984712181 0.997600070100712" />
-    <limit
-      lower="-0.9"
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