Commit message: Modified the URDF file for the right ros2 control.

File: gazebo_2_sim_pid/urdf/link2_urdf.urdf.xacro (robot description, xacro)
@@ -164,26 +164,21 @@
       velocity="0.3" />
   </joint>
+ <!-- ROS2_CONTROL CONFIGURATION -->
   <ros2_control name="GazeboSystem" type="system">
-    <hardware>
-      <plugin>gazebo_ros2_control/GazeboSystem</plugin>
-    </hardware>
-    <joint name="joint_1">
-      <command_interface name="position">
-      </command_interface>
-      <state_interface name="position">
-        <param name="initial_value">0</param>
-      </state_interface>
-      <state_interface name="velocity"/>
-      <state_interface name="effort"/>
-    </joint>
-    <joint name="joint_2">
-      <command_interface name="position">
-      </command_interface>
-      <state_interface name="position">
-        <param name="initial_value">0</param>
-      </state_interface>
-      <state_interface name="velocity"/>
-      <state_interface name="effort"/>
-    </joint>
+      <hardware>
+          <plugin>gazebo_ros2_control/GazeboSystem</plugin>
+      </hardware>
+      <joint name="joint_1">
+          <command_interface name="effort" />
+          <state_interface name="position" />
+          <state_interface name="velocity" />
+          <state_interface name="effort" />
+      </joint>
+      <joint name="joint_2">
+          <command_interface name="effort" />
+          <state_interface name="position" />
+          <state_interface name="velocity" />
+          <state_interface name="effort" />
+      </joint>
   </ros2_control>
   <gazebo>
